File: cardV2.sch (EAGLE design)
At the start: 48 parts, among them IC1 ATTINY1616, IC2 LTC1992-1, IC3 LTC1992, IC4 LTC6911, IC5 LTC2402, SW1 SPST_TACT-EVQQ2, SW2 SPST_TACT-EVQQ2, SW3 SPST_TACT-EVQQ2, SW4 SPST_TACT-EVQQ2

Commit message: Small changes in board V2 & more test in programming
BTW the programm works, the problem came from the not well connected LCD
Parts:
- added CLK, CS_A, CS_S, D/C, GA, GB, MISO, MOSI, RST, VA, VA+, VA-, VB, VB+, VB-, VCAP: TPSQB1,27, testpad:TPSQB1,27
Connections:
- net CLK: now also CLK.TP
- net D/C: now also D/C.TP
- net MISO: now also MISO.TP
- net MOSI: now also MOSI.TP
- net N$16: now also VA-.TP
- net N$17: now also VA+.TP
- net N$25: now also VB-.TP
- net N$26: now also VB+.TP
- net N$29: now also GB.TP
- net N$3: now also VCAP.TP
- net N$37: now also GA.TP
- net RAWA: now also VA.TP
- net RAWB: now also VB.TP
- net RST: now also RST.TP
- net _CS_ADC: now also CS_A.TP
- net _CS_SCR: now also CS_S.TP
Changed lines of the file:
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@@
 <part name="GND24" library="supply1" deviceset="GND" device=""/>
 <part name="PIN" library="con-amp" deviceset="MTA03-100" device=""/>
+<part name="VA+" library="testpad" deviceset="TPSQ" device="B1,27" value="TPSQB1,27"/>
+<part name="VA-" library="testpad" deviceset="TPSQ" device="B1,27" value="TPSQB1,27"/>
+<part name="VB+" library="testpad" deviceset="TPSQ" device="B1,27" value="TPSQB1,27"/>
+<part name="VB-" library="testpad" deviceset="TPSQ" device="B1,27" value="TPSQB1,27"/>
+<part name="VA" library="testpad" deviceset="TPSQ" device="B1,27" value="TPSQB1,27"/>
+<part name="VB" library="testpad" deviceset="TPSQ" device="B1,27" value="TPSQB1,27"/>
+<part name="GA" library="testpad" deviceset="TPSQ" device="B1,27" value="TPSQB1,27"/>
+<part name="GB" library="testpad" deviceset="TPSQ" device="B1,27" value="TPSQB1,27"/>
+<part name="VCAP" library="testpad" deviceset="TPSQ" device="B1,27" value="TPSQB1,27"/>
+<part name="CLK" library="testpad" deviceset="TPSQ" device="B1,27" value="TPSQB1,27"/>
+<part name="MISO" library="testpad" deviceset="TPSQ" device="B1,27" value="TPSQB1,27"/>
+<part name="MOSI" library="testpad" deviceset="TPSQ" device="B1,27" value="TPSQB1,27"/>
+<part name="CS_A" library="testpad" deviceset="TPSQ" device="B1,27" value="TPSQB1,27"/>
+<part name="CS_S" library="testpad" deviceset="TPSQ" device="B1,27" value="TPSQB1,27"/>
+<part name="D/C" library="testpad" deviceset="TPSQ" device="B1,27" value="TPSQB1,27"/>
+<part name="RST" library="testpad" deviceset="TPSQ" device="B1,27" value="TPSQB1,27"/>
 </parts>
 <sheets>
@@
 <instance part="GND24" gate="1" x="-83.82" y="190.5"/>
 <instance part="PIN" gate="G$1" x="-114.3" y="66.04" rot="R90"/>
+<instance part="VA+" gate="G$1" x="-195.58" y="134.62" rot="R180"/>
+<instance part="VA-" gate="G$1" x="-195.58" y="109.22"/>
+<instance part="VB+" gate="G$1" x="-195.58" y="53.34" rot="R180"/>
+<instance part="VB-" gate="G$1" x="-195.58" y="27.94"/>
+<instance part="VA" gate="G$1" x="-177.8" y="137.16" rot="R180"/>
+<instance part="VB" gate="G$1" x="-177.8" y="55.88" rot="R180"/>
+<instance part="GA" gate="G$1" x="-78.74" y="134.62" rot="R180"/>
+<instance part="GB" gate="G$1" x="-78.74" y="114.3"/>
+<instance part="VCAP" gate="G$1" x="-30.48" y="76.2" rot="R180"/>
+<instance part="CLK" gate="G$1" x="-58.42" y="180.34" rot="R180"/>
+<instance part="MISO" gate="G$1" x="-50.8" y="180.34" rot="R180"/>
+<instance part="MOSI" gate="G$1" x="-43.18" y="180.34" rot="R180"/>
+<instance part="CS_A" gate="G$1" x="-35.56" y="180.34" rot="R180"/>
+<instance part="CS_S" gate="G$1" x="-27.94" y="180.34" rot="R180"/>
+<instance part="D/C" gate="G$1" x="-15.24" y="180.34" rot="R180"/>
+<instance part="RST" gate="G$1" x="-5.08" y="180.34" rot="R180"/>
 </instances>
 <busses>
@@
 <wire x1="-30.48" y1="71.12" x2="-20.32" y2="71.12" width="0.1524" layer="91"/>
 <wire x1="-20.32" y1="71.12" x2="-20.32" y2="58.42" width="0.1524" layer="91"/>
+<pinref part="VCAP" gate="G$1" pin="TP"/>
+<wire x1="-30.48" y1="73.66" x2="-30.48" y2="71.12" width="0.1524" layer="91"/>
+<junction x="-30.48" y="71.12"/>
 </segment>
 </net>
@@
 <label x="-60.96" y="66.04" size="1.778" layer="95" xref="yes"/>
 </segment>
+<segment>
+<pinref part="D/C" gate="G$1" pin="TP"/>
+<wire x1="-15.24" y1="175.26" x2="-15.24" y2="177.8" width="0.1524" layer="91"/>
+<label x="-15.24" y="175.26" size="1.778" layer="95" rot="R270" xref="yes"/>
+</segment>
 </net>
 <net name="MOSI" class="0">
@@
 <wire x1="-73.66" y1="71.12" x2="-60.96" y2="71.12" width="0.1524" layer="91"/>
 </segment>
+<segment>
+<pinref part="MOSI" gate="G$1" pin="TP"/>
+<wire x1="-43.18" y1="175.26" x2="-43.18" y2="177.8" width="0.1524" layer="91"/>
+<label x="-43.18" y="175.26" size="1.778" layer="95" rot="R270" xref="yes"/>
+</segment>
 </net>
 <net name="_CS_SCR" class="0">
@@
 <label x="-60.96" y="60.96" size="1.778" layer="95" xref="yes"/>
 </segment>
+<segment>
+<pinref part="CS_S" gate="G$1" pin="TP"/>
+<wire x1="-27.94" y1="175.26" x2="-27.94" y2="177.8" width="0.1524" layer="91"/>
+<label x="-27.94" y="175.26" size="1.778" layer="95" rot="R270" xref="yes"/>
+</segment>
 </net>
 <net name="RST" class="0">
@@
 <wire x1="-73.66" y1="63.5" x2="-68.58" y2="63.5" width="0.1524" layer="91"/>
 <label x="-68.58" y="63.5" size="1.778" layer="95" xref="yes"/>
+</segment>
+<segment>
+<pinref part="RST" gate="G$1" pin="TP"/>
+<wire x1="-5.08" y1="175.26" x2="-5.08" y2="177.8" width="0.1524" layer="91"/>
+<label x="-5.08" y="175.26" size="1.778" layer="95" rot="R270" xref="yes"/>
 </segment>
 </net>
@@
 <wire x1="-215.9" y1="114.3" x2="-213.36" y2="114.3" width="0.1524" layer="91"/>
 <wire x1="-195.58" y1="114.3" x2="-213.36" y2="114.3" width="0.1524" layer="91"/>
+<pinref part="VA-" gate="G$1" pin="TP"/>
+<wire x1="-195.58" y1="114.3" x2="-195.58" y2="111.76" width="0.1524" layer="91"/>
+<junction x="-195.58" y="114.3"/>
 </segment>
 </net>
@@
 <wire x1="-177.8" y1="132.08" x2="-170.18" y2="132.08" width="0.1524" layer="91"/>
 <label x="-170.18" y="132.08" size="1.778" layer="95" xref="yes"/>
+<pinref part="VA" gate="G$1" pin="TP"/>
+<wire x1="-177.8" y1="134.62" x2="-177.8" y2="132.08" width="0.1524" layer="91"/>
+<junction x="-177.8" y="132.08"/>
 </segment>
 <segment>
@@
 <label x="-167.64" y="50.8" size="1.778" layer="95" xref="yes"/>
 <pinref part="IC3" gate="G$1" pin="-OUT"/>
+<junction x="-177.8" y="50.8"/>
+<pinref part="VB" gate="G$1" pin="TP"/>
+<wire x1="-177.8" y1="50.8" x2="-177.8" y2="53.34" width="0.1524" layer="91"/>
 </segment>
 <segment>
@@
 <pinref part="IC5" gate="G$1" pin="CH0"/>
 <wire x1="-78.74" y1="121.92" x2="-66.04" y2="121.92" width="0.1524" layer="91"/>
+<pinref part="GB" gate="G$1" pin="TP"/>
+<wire x1="-78.74" y1="119.38" x2="-78.74" y2="116.84" width="0.1524" layer="91"/>
+<junction x="-78.74" y="119.38"/>
 </segment>
 </net>
@@
 <pinref part="IC4" gate="G$1" pin="OUTA"/>
 <wire x1="-78.74" y1="129.54" x2="-83.82" y2="129.54" width="0.1524" layer="91"/>
+<pinref part="GA" gate="G$1" pin="TP"/>
+<wire x1="-78.74" y1="129.54" x2="-78.74" y2="132.08" width="0.1524" layer="91"/>
+<junction x="-78.74" y="129.54"/>
 </segment>
 </net>
@@
 <wire x1="-60.96" y1="76.2" x2="-73.66" y2="76.2" width="0.1524" layer="91"/>
 </segment>
+<segment>
+<pinref part="CLK" gate="G$1" pin="TP"/>
+<wire x1="-58.42" y1="175.26" x2="-58.42" y2="177.8" width="0.1524" layer="91"/>
+<label x="-58.42" y="175.26" size="1.778" layer="95" rot="R270" xref="yes"/>
+</segment>
 </net>
 <net name="MISO" class="0">
@@
 <label x="-68.58" y="73.66" size="1.778" layer="95" xref="yes"/>
 </segment>
+<segment>
+<pinref part="MISO" gate="G$1" pin="TP"/>
+<wire x1="-50.8" y1="175.26" x2="-50.8" y2="177.8" width="0.1524" layer="91"/>
+<label x="-50.8" y="175.26" size="1.778" layer="95" rot="R270" xref="yes"/>
+</segment>
 </net>
 <net name="_CS_ADC" class="0">
@@
 <wire x1="-73.66" y1="58.42" x2="-60.96" y2="56.642" width="0.1524" layer="91"/>
 <label x="-60.96" y="56.642" size="1.778" layer="95" xref="yes"/>
+</segment>
+<segment>
+<pinref part="CS_A" gate="G$1" pin="TP"/>
+<wire x1="-35.56" y1="175.26" x2="-35.56" y2="177.8" width="0.1524" layer="91"/>
+<label x="-35.56" y="175.26" size="1.778" layer="95" rot="R270" xref="yes"/>
 </segment>
 </net>
@@
 <wire x1="-195.58" y1="124.46" x2="-193.04" y2="124.46" width="0.1524" layer="91"/>
 <wire x1="-213.36" y1="129.54" x2="-195.58" y2="129.54" width="0.1524" layer="91"/>
+<pinref part="VA+" gate="G$1" pin="TP"/>
+<wire x1="-195.58" y1="129.54" x2="-195.58" y2="132.08" width="0.1524" layer="91"/>
+<junction x="-195.58" y="129.54"/>
 </segment>
 </net>
@@
 <pinref part="IC3" gate="G$1" pin="-IN"/>
 <wire x1="-213.36" y1="33.02" x2="-195.58" y2="33.02" width="0.1524" layer="91"/>
+<junction x="-195.58" y="33.02"/>
+<pinref part="VB-" gate="G$1" pin="TP"/>
+<wire x1="-195.58" y1="30.48" x2="-195.58" y2="33.02" width="0.1524" layer="91"/>
 </segment>
 </net>
@@
 <pinref part="IC3" gate="G$1" pin="+IN"/>
 <wire x1="-213.36" y1="48.26" x2="-195.58" y2="48.26" width="0.1524" layer="91"/>
-</segment>
-</net>
+<junction x="-195.58" y="48.26"/>
+<pinref part="VB+" gate="G$1" pin="TP"/>
+<wire x1="-195.58" y1="48.26" x2="-195.58" y2="50.8" width="0.1524" layer="91"/>
+</segment>
+</net>

Commit message: Completly separated power lines (analog vs digital)
And more program tests
Parts:
- added SJ1, SJ2: (no value), jumper:SJ
Connections:
- new net AGND: AMPA-2.1, AMPB-2.1, C2.1.2, C2.2, C3.1.2, C3.2, C4.1.-, C4.2, IC2P.VEE, IC3P.VEE, IC4.V-, IC5.ZSET, R24.2, R34.2, SJ1.2, VOLTA-2.1, VOLTB-2.1
- new net V+: C2.1, C3.1, C4.1, IC2P.VDD, IC3P.VDD, IC4.V+, IC5.FSET, R29.2, R39.2, SJ2.2
- net +3V3: now also SJ2.1; no longer C2.1, C3.1, C4.1, IC2P.VDD, IC3P.VDD, IC4.V+, IC5.FSET, R29.2, R39.2
- net GND: now also SJ1.1; no longer AMPA-2.1, AMPB-2.1, C2.1.2, C2.2, C3.1.2, C3.2, C4.1.-, C4.2, IC2P.VEE, IC3P.VEE, IC4.V-, IC5.ZSET, R24.2, R34.2, VOLTA-2.1, VOLTB-2.1
