File: cardV3.brd (EAGLE design)
At the start: 83.5 x 52.2 mm, 66 parts, among them IC1 ATTINY1616, IC2 LTC1992-1, IC3 LTC1992, IC4 LTC6911, IC5 LTC2402, SW1 SPST_TACT-EVQQ2, SW2 SPST_TACT-EVQQ2, SW3 SPST_TACT-EVQQ2, SW4 SPST_TACT-EVQQ2

Commit message: Better V3...
Parts:
- removed C2.1, C3.1: 1u, resistor:C0805
- removed C4.1: 1u, adafruit:A/3216-18R
- removed GA, GB: TPSQB1,27, testpad:B1,27
- removed IC5: LTC2402, HomeMade:MSOP10
- removed PIN: (no value), con-amp:10X03MTA
- removed R21, R22, R31, R32: 470k, resistor:M0805
- removed R23, R33: 10k, resistor:M0805
- removed R24, R34: 1, resistor:M0805
- removed R29, R39: 100, resistor:M0805
- removed RESA, RESB: (no value), con-phoenix-254:2POL254
- removed SJ1, SJ2: (no value), jumper:SJ
- added GAN, VAN: (no value), jumper:SJ
- added PA7: TPSQB1,27, testpad:B1,27
- added R1A, R1B, R2A, R2B: 1M, resistor:M0805
- added R3A, R3B, R4A, R4B: 390k, resistor:M0805
- added R5A, R5B, R6A, R6B: 100k, resistor:M0805
- added RA, RB: 1, resistor:M0805
- IC2: value LTC1992-1 -> AD8231; device linear-technology-2:MSOP8 -> HomeMade:LFCSP16
- IC3: value LTC1992 -> AD8231; device linear-technology-2:MSOP8 -> HomeMade:LFCSP16
- IC4: value LTC6911 -> LTC2402
- moved C2 22.7 mm to (16.8, 47.0), turned to 270 degrees
- moved IC2 19.8 mm to (14.0, 46.8), turned to 0 degrees
- moved VB- 19.5 mm to (10.0, 33.1)
- moved VA- 18.1 mm to (10.8, 50.2)
- moved VA 17.1 mm to (17.1, 44.3)
- moved C3 16.6 mm to (16.9, 27.4), flipped to the bottom, turned to 270 degrees
- moved IC3 15.6 mm to (14.0, 28.6), flipped to the top, turned to 0 degrees
- moved VB+ 14.2 mm to (9.84, 25.2), turned to 180 degrees
- moved VA+ 11.3 mm to (9.84, 43.7), turned to 180 degrees
- moved IC4 7.10 mm to (19.7, 22.2)
- moved C5 6.25 mm to (21.3, 22.2)
- moved C4 4.61 mm to (16.7, 23.2), flipped to the bottom, turned to 270 degrees
- moved VOLTA 4.49 mm to (3.17, 47.0)
- moved AMPA 3.24 mm to (3.17, 39.4)
- moved MISO 2.95 mm to (24.3, 16.0)
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- renumbered U$1 to SCR
Connections:
- removed net G0: IC1.2, IC4.4
- removed net G1: IC1.3, IC4.5
- removed net G2: IC1.4, IC4.6
- removed net N$21: C2.1.1, IC2.2, IC2.7
- removed net N$22: R21.2, R22.1
- removed net N$25: AMPB.1, IC3.1, R33.2, R34.1, VB-.TP
- removed net N$26: IC3.8, R32.2, R33.1, RESB.1, VB+.TP
- removed net N$27: R21.1, VOLTA.1
- removed net N$28: R29.1, RESA.2
- removed net N$29: GB.TP, IC4.8, IC5.4
- removed net N$31: C3.1.1, IC3.2, IC3.7
- removed net N$32: R31.2, R32.1
- removed net N$35: R31.1, VOLTB.1
- removed net N$36: R39.1, RESB.2
- removed net N$37: GA.TP, IC4.10, IC5.3
- removed net RAWA: IC2.5, IC4.1, VA.TP
- removed net RAWB: IC3.5, IC4.3, VB.TP
- new net A0: IC1.2, IC2.14, IC3.14
- new net A1: IC1.3, IC2.15, IC3.15
- new net A2: IC1.4, IC2.16, IC3.16
- new net N$10: IC2.6, R5A.1, R6A.2
- new net N$11: R3A.1, VOLTA.2
- new net N$12: AMPA.2, IC2.2, R1A.2, R3A.2, RA.1, VA-.TP
- new net N$13: IC2.7, IC2.8, IC2.9
- new net N$14: AMPA.1, IC2.3, R2A.1, R4A.2, RA.2, VA+.TP
- new net N$15: R3B.1, VOLTB.2
- new net N$19: IC1.5, PA7.TP
- new net VA: IC2.10, IC4.3, VA.TP
- new net VB: IC3.10, IC4.4, VB.TP
- new net _CS_INA: IC1.6, IC2.13
- new net _CS_INB: IC1.7, IC3.13
- net +3V3: now also IC4.1, IC4.10, VAN.1; no longer IC5.1, IC5.10, SJ2.1
- net AGND: now also GAN.2, IC2.11, IC2.17, IC3.11, IC3.17, IC4.5, R1A.1, R1B.1, R2A.2, R2B.2, R5A.2, R5B.2; no longer AMPA.2, AMPB.2, C2.1.2, C3.1.2, C4.1.-, IC2.6, IC3.6, IC4.9, IC5.5, R24.2, R34.2, SJ1.2, VOLTA.2, VOLTB.2
- net CLK: now also IC4.9; no longer IC5.9
- net GND: now also GAN.1, IC4.6; no longer IC5.6, SJ1.1
- net MISO: now also IC4.8; no longer IC5.8
- net N$16: now also IC3.7, IC3.8, IC3.9; no longer AMPA.1, IC2.1, R23.2, R24.1, VA-.TP
- net N$17: now also R4B.1, VOLTB.1; no longer IC2.8, R22.2, R23.1, RESA.1, VA+.TP
- net N$18: now also IC3.6, R5B.1, R6B.2; no longer C4.1.+, IC4.2
- net N$7: now also R4A.1, VOLTA.1; no longer IC1.7, PIN.1
- net N$8: now also AMPB.2, IC3.2, R1B.2, R3B.2, RB.1, VB-.TP; no longer IC1.5, PIN.3
- net N$9: now also AMPB.1, IC3.3, R2B.1, R4B.2, RB.2, VB+.TP; no longer IC1.6, PIN.2
- net V+: now also IC2.12, IC2.5, IC3.12, IC3.5, IC4.2, R6A.1, R6B.1, VAN.2; no longer IC2.3, IC3.3, IC4.7, IC5.2, R29.2, R39.2, SJ2.2
- net _CS_ADC: now also IC4.7; no longer IC5.7
Routing:
- net A2: track 0.00 -> 69.8 mm, vias 0 -> 3
- net A1: track 0.00 -> 66.9 mm, vias 0 -> 3
- net A0: track 0.00 -> 64.6 mm, vias 0 -> 3
- net _CS_INA: track 0.00 -> 64.3 mm, vias 0 -> 2
- net N$26: track 47.3 -> 0.00 mm, vias 1 -> 0
- net _CS_INB: track 0.00 -> 44.9 mm, vias 0 -> 2
- net VA: track 0.00 -> 29.3 mm, vias 0 -> 2
- net N$17: track 30.8 -> 2.86 mm
- net N$12: track 0.00 -> 27.7 mm, vias 0 -> 1
- net N$7: track 28.5 -> 2.86 mm, vias 1 -> 0
- net AGND: track 160.3 -> 136.1 mm, vias 5 -> 31
- net G0: track 20.7 -> 0.00 mm
- net N$14: track 0.00 -> 20.2 mm
- net G1: track 20.1 -> 0.00 mm
- net G2: track 19.9 -> 0.00 mm
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
Commit message: improvement
Parts:
- added C7: (no value), rcl:153CLV-0405
- moved VCAP 2.81 mm to (56.5, 49.1)
- moved ON/OFF 2.54 mm to (41.9, 49.5)
Connections:
- net +3V3: now also C7.+
- net GND: now also C7.-
Routing:
- net +3V3: track 217.3 -> 227.4 mm, vias 6 -> 7
- net GND: track 250.1 -> 257.5 mm
- net N$1: track 14.9 -> 12.3 mm
