File: eagle/cardV3.brd (EAGLE design)
At the start: 83.5 x 52.2 mm, 63 parts, among them IC1 ATTINY1616, IC2 AD8231, IC3 AD8231, IC4 LTC2402, SW1 SPST_TACT-EVQQ2, SW2 SPST_TACT-EVQQ2, SW3 SPST_TACT-EVQQ2, SW4 SPST_TACT-EVQQ2

Commit message: Restructured repo
Parts:
- removed PROG: (no value), con-amp:10X03MTA
- added X1: 1501_03, con-lumberg:1501_03
Connections:
- net +3V3: now also X1.3; no longer PROG.1
- net GND: now also X1.1; no longer PROG.3
- net UPDI: now also X1.2; no longer PROG.2
Routing:
- net GND: track 257.5 -> 264.7 mm
- net +3V3: track 227.4 -> 223.4 mm
- net UPDI: track 36.8 -> 33.7 mm
