File: eagle/cardV3.sch (EAGLE design)
At the start: 63 parts, among them IC1 ATTINY1616, IC2 AD8231, IC3 AD8231, IC4 LTC2402, SW1 SPST_TACT-EVQQ2, SW2 SPST_TACT-EVQQ2, SW3 SPST_TACT-EVQQ2, SW4 SPST_TACT-EVQQ2

Commit message: Restructured repo
Parts:
- removed PROG: (no value), con-amp:MTA03-100
- added X1: 1501_03, con-lumberg:1501_03
Connections:
- net +3V3: now also X1.3; no longer PROG.1
- net GND: now also X1.1; no longer PROG.3
- net UPDI: now also X1.2; no longer PROG.2
Changed lines of the file:
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@@
 <part name="+3V16" library="supply1" deviceset="+3V3" device=""/>
 <part name="GND23" library="supply1" deviceset="GND" device=""/>
-<part name="PROG" library="con-amp" deviceset="MTA03-100" device=""/>
 <part name="+3V17" library="supply1" deviceset="+3V3" device=""/>
 <part name="GND24" library="supply1" deviceset="GND" device=""/>
@@
 <part name="+3V8" library="supply1" deviceset="+3V3" device=""/>
 <part name="GND5" library="supply1" deviceset="GND" device=""/>
+<part name="X1" library="con-lumberg" deviceset="1501_03" device=""/>
 </parts>
 <sheets>
@@
 <instance part="+3V16" gate="G$1" x="137.16" y="86.36"/>
 <instance part="GND23" gate="1" x="137.16" y="73.66"/>
-<instance part="PROG" gate="G$1" x="147.32" y="198.12"/>
-<instance part="+3V17" gate="G$1" x="139.7" y="195.58"/>
-<instance part="GND24" gate="1" x="149.86" y="187.96"/>
+<instance part="+3V17" gate="G$1" x="147.32" y="190.5" rot="R180"/>
+<instance part="GND24" gate="1" x="152.4" y="187.96"/>
 <instance part="VA+" gate="G$1" x="50.8" y="111.76"/>
 <instance part="VA-" gate="G$1" x="50.8" y="132.08" rot="R180"/>
@@
 <instance part="+3V8" gate="G$1" x="127" y="203.2"/>
 <instance part="GND5" gate="1" x="127" y="182.88"/>
+<instance part="X1" gate="G$1" x="149.86" y="203.2" rot="R90"/>
 </instances>
 <busses>
@@
 </segment>
 <segment>
-<pinref part="PROG" gate="G$1" pin="1"/>
-<wire x1="144.78" y1="195.58" x2="144.78" y2="190.5" width="0.1524" layer="91"/>
-<pinref part="+3V17" gate="G$1" pin="+3V3"/>
-<wire x1="144.78" y1="190.5" x2="139.7" y2="190.5" width="0.1524" layer="91"/>
-<wire x1="139.7" y1="190.5" x2="139.7" y2="193.04" width="0.1524" layer="91"/>
-</segment>
-<segment>
 <pinref part="+3V18" gate="G$1" pin="+3V3"/>
 <pinref part="VAN" gate="1" pin="1"/>
@@
 <pinref part="+3V8" gate="G$1" pin="+3V3"/>
 <wire x1="127" y1="200.66" x2="127" y2="195.58" width="0.1524" layer="91"/>
+</segment>
+<segment>
+<pinref part="X1" gate="G$1" pin="3"/>
+<pinref part="+3V17" gate="G$1" pin="+3V3"/>
+<wire x1="147.32" y1="193.04" x2="147.32" y2="198.12" width="0.1524" layer="91"/>
 </segment>
 </net>
@@
 </segment>
 <segment>
-<pinref part="PROG" gate="G$1" pin="3"/>
 <pinref part="GND24" gate="1" pin="GND"/>
-<wire x1="149.86" y1="195.58" x2="149.86" y2="190.5" width="0.1524" layer="91"/>
+<wire x1="152.4" y1="198.12" x2="152.4" y2="190.5" width="0.1524" layer="91"/>
+<pinref part="X1" gate="G$1" pin="1"/>
 </segment>
 <segment>
@@
 </segment>
 <segment>
-<pinref part="PROG" gate="G$1" pin="2"/>
-<wire x1="147.32" y1="195.58" x2="147.32" y2="187.96" width="0.1524" layer="91"/>
-<wire x1="147.32" y1="187.96" x2="144.78" y2="187.96" width="0.1524" layer="91"/>
-<label x="144.78" y="187.96" size="1.778" layer="95" rot="R180" xref="yes"/>
-</segment>
-</net>
+<wire x1="144.78" y1="190.5" x2="142.24" y2="190.5" width="0.1524" layer="91"/>
+<label x="142.24" y="190.5" size="1.778" layer="95" rot="R180" xref="yes"/>
+<pinref part="X1" gate="G$1" pin="2"/>
+<wire x1="144.78" y1="190.5" x2="144.78" y2="198.12" width="0.1524" layer="91"/>
+</segment>
+</net>
