File: kicad/cardV4.kicad_pcb (KiCad board)
At the start: 2 copper layers, 79.9 x 68.7 mm, 74 parts, among them J1 Charge, J10 AOP, J11 Volt1, J12 Volt2, J13 Amp, J14 Res, J20 UPDI, SW00 ON/OFF, SW1 SW_Push, SW2 SW_Push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

Commit message: Schematic for V5
Parts:
- TP10, TP11, TP12, TP130, TP131, TP14, TP20, TP21, TP210, TP22, TP23, TP24, TP25, TP26, TP27, TP28, TP29, TP30: footprint perso:Probing_pad -> telec:Probing_pad
- U30: footprint perso:NOKIA_3310_LCD -> telec:NOKIA_3310_LCD
Changed lines of the file:
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@@
     )
   )
-  (module perso:NOKIA_3310_LCD (layer F.Cu)
+  (module telec:NOKIA_3310_LCD (layer F.Cu)
     (at 68.961 16.764)
     (fp_text reference U30 (at 5.588 2.413 90) (layer F.SilkS)
@@
     (pad "" thru_hole circle (at -17.25 6) (size 2 2) (drill 2) (layers *.Cu))
   )
-  (module perso:Probing_pad (layer F.Cu)
+  (module telec:Probing_pad (layer F.Cu)
     (at 44.196 37.465)
     (fp_text reference TP26 (at 0 4.826 90) (layer F.SilkS)
@@
     )
   )
-  (module perso:Probing_pad (layer F.Cu)
+  (module telec:Probing_pad (layer F.Cu)
     (at 42.164 38.989)
     (fp_text reference TP210 (at 0 5.461 90) (layer F.SilkS)
@@
     )
   )
-  (module perso:Probing_pad (layer F.Cu)
+  (module telec:Probing_pad (layer F.Cu)
     (at 13.97 31.242)
     (fp_text reference TP10 (at 2.667 1.905) (layer F.SilkS)
@@
       (net 6 GNDREF))
   )
-  (module perso:Probing_pad (layer F.Cu)
+  (module telec:Probing_pad (layer F.Cu)
     (at 20.32 35.052)
     (fp_text reference TP11 (at 0.762 0.254) (layer F.SilkS)
@@
       (net 29 /V1))
   )
-  (module perso:Probing_pad (layer F.Cu)
+  (module telec:Probing_pad (layer F.Cu)
     (at 20.32 27.432)
     (fp_text reference TP12 (at 0.889 0.254) (layer F.SilkS)
@@
       (net 30 /V2))
   )
-  (module perso:Probing_pad (layer F.Cu)
+  (module telec:Probing_pad (layer F.Cu)
     (at 20.32 15.621)
     (fp_text reference TP14 (at 2.921 2.159) (layer F.SilkS)
@@
       (net 20 /R))
   )
-  (module perso:Probing_pad (layer F.Cu)
+  (module telec:Probing_pad (layer F.Cu)
     (at 35.306 41.91)
     (fp_text reference TP20 (at 0 4.826 90) (layer F.SilkS)
@@
       (net 39 /CLK))
   )
-  (module perso:Probing_pad (layer F.Cu)
+  (module telec:Probing_pad (layer F.Cu)
     (at 39.878 40.005)
     (fp_text reference TP21 (at 0 4.699 90) (layer F.SilkS)
@@
       (net 40 /MISO))
   )
-  (module perso:Probing_pad (layer F.Cu)
+  (module telec:Probing_pad (layer F.Cu)
     (at 37.465 40.894)
     (fp_text reference TP22 (at 0 4.699 90) (layer F.SilkS)
@@
       (net 41 /MOSI))
   )
-  (module perso:Probing_pad (layer F.Cu)
+  (module telec:Probing_pad (layer F.Cu)
     (at 28.194 40.767)
     (fp_text reference TP23 (at 0 4.826 90) (layer F.SilkS)
@@
       (net 42 /~ADC_CS))
   )
-  (module perso:Probing_pad (layer F.Cu)
+  (module telec:Probing_pad (layer F.Cu)
     (at 46.101 35.56)
     (fp_text reference TP24 (at 0 4.953 90) (layer F.SilkS)
@@
       (net 43 /~SCR_CS))
   )
-  (module perso:Probing_pad (layer F.Cu)
+  (module telec:Probing_pad (layer F.Cu)
     (at 31.242 41.91)
     (fp_text reference TP25 (at 0 4.826 90) (layer F.SilkS)
@@
       (net 44 /~ADC_RST))
   )
-  (module perso:Probing_pad (layer F.Cu)
+  (module telec:Probing_pad (layer F.Cu)
     (at 27.686 38.481)
     (fp_text reference TP27 (at -1.143 4.572 90) (layer F.SilkS)
@@
       (net 22 /~STANDBY))
   )
-  (module perso:Probing_pad (layer F.Cu)
+  (module telec:Probing_pad (layer F.Cu)
     (at 30.353 39.751)
     (fp_text reference TP28 (at -0.762 4.953 90) (layer F.SilkS)
@@
       (net 27 /~RDY))
   )
-  (module perso:Probing_pad (layer F.Cu)
+  (module telec:Probing_pad (layer F.Cu)
     (at 33.274 40.513)
     (fp_text reference TP29 (at 0 4.826 90) (layer F.SilkS)
@@
       (net 24 /~SYNC))
   )
-  (module perso:Probing_pad (layer F.Cu)
+  (module telec:Probing_pad (layer F.Cu)
     (at 66.04 11.557)
     (fp_text reference TP30 (at 3.048 2.032) (layer F.SilkS)
@@
       (net 10 "Net-(C31-Pad1)"))
   )
-  (module perso:Probing_pad (layer F.Cu)
+  (module telec:Probing_pad (layer F.Cu)
     (at 20.32 20.828)
     (fp_text reference TP130 (at 3.429 2.032) (layer F.SilkS)
@@
       (net 19 /I+))
   )
-  (module perso:Probing_pad (layer F.Cu)
+  (module telec:Probing_pad (layer F.Cu)
     (at 20.32 17.78)
     (fp_text reference TP131 (at 3.429 2.032) (layer F.SilkS)
