File: kicad/cardV4.sch (KiCad schematic (older format))
At the start: 74 parts, among them J1 Charge, J10 AOP, J11 Volt1, J12 Volt2, J13 Amp, J14 Res, J20 UPDI, SW00 ON/OFF, SW1 SW_Push, SW2 SW_Push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

Commit message: Schematic for V5
Parts:
- TP10, TP11, TP12, TP130, TP131, TP14, TP20, TP21, TP210, TP22, TP23, TP24, TP25, TP26, TP27, TP28, TP29, TP30: footprint perso:Probing_pad -> telec:Probing_pad
- U02: symbol perso:ADR291GT9Z -> telec:ADR291GT9Z
- U10: symbol perso:LT1178 -> telec:LT1178
- U12: symbol perso:AD7731 -> telec:AD7731
- U20: symbol perso:ATtiny1616 -> telec:ATtiny1616
- U30: footprint perso:NOKIA_3310_LCD -> telec:NOKIA_3310_LCD; symbol perso:Nokia_3310_LCD -> telec:Nokia_3310_LCD
Changed lines of the file:
@@
 EESchema Schematic File Version 4
-LIBS:cardV4-cache
-EELAYER 26 0
+EELAYER 30 0
 EELAYER END
 $Descr A4 11693 8268
@@
 $EndComp
 $Comp
-L perso:AD7731 U12
+L telec:AD7731 U12
 U 1 1 5C168DFB
 P 3550 4600
@@
 $EndComp
 $Comp
-L perso:LT1178 U10
+L telec:LT1178 U10
 U 1 1 5C16AE7D
 P 2450 2600
@@
 $EndComp
 $Comp
-L perso:LT1178 U10
+L telec:LT1178 U10
 U 3 1 5C16B184
 P 1250 2550
@@
 Connection ~ 1400 2800
 $Comp
-L perso:ATtiny1616 U20
+L telec:ATtiny1616 U20
 U 1 1 5C1BF9FF
 P 7100 4300
@@
 $EndComp
 $Comp
-L perso:Nokia_3310_LCD U30
+L telec:Nokia_3310_LCD U30
 U 1 1 5C1BFA9E
 P 9600 4000
 F 0 "U30" H 10050 4050 60  0000 L CNN
 F 1 "Nokia_3310_LCD" H 9250 2800 60  0000 L CNN
-F 2 "perso:NOKIA_3310_LCD" H 10328 3376 60  0001 L CNN
+F 2 "telec:NOKIA_3310_LCD" H 10328 3376 60  0001 L CNN
 F 3 "" V 9600 3850 60  0000 C CNN
 	1    9600 4000
@@
 F 0 "TP30" H 8958 3470 50  0000 L CNN
 F 1 "Vcap" H 8958 3379 50  0000 L CNN
-F 2 "perso:Probing_pad" H 9100 3350 50  0001 C CNN
+F 2 "telec:Probing_pad" H 9100 3350 50  0001 C CNN
 F 3 "~" H 9100 3350 50  0001 C CNN
 	1    8900 3350
@@
 F 0 "TP11" H 1958 4220 50  0000 L CNN
 F 1 "V1" H 1958 4129 50  0000 L CNN
-F 2 "perso:Probing_pad" H 2100 4100 50  0001 C CNN
+F 2 "telec:Probing_pad" H 2100 4100 50  0001 C CNN
 F 3 "~" H 2100 4100 50  0001 C CNN
 	1    1900 4100
@@
 F 0 "TP12" H 1958 4720 50  0000 L CNN
 F 1 "V2" H 1958 4629 50  0000 L CNN
-F 2 "perso:Probing_pad" H 2100 4600 50  0001 C CNN
+F 2 "telec:Probing_pad" H 2100 4600 50  0001 C CNN
 F 3 "~" H 2100 4600 50  0001 C CNN
 	1    1900 4600
@@
 F 0 "TP130" H 1958 5220 50  0000 L CNN
 F 1 "I+" H 1958 5129 50  0000 L CNN
-F 2 "perso:Probing_pad" H 2100 5100 50  0001 C CNN
+F 2 "telec:Probing_pad" H 2100 5100 50  0001 C CNN
 F 3 "~" H 2100 5100 50  0001 C CNN
 	1    1900 5100
@@
 F 0 "TP131" H 1958 5520 50  0000 L CNN
 F 1 "I-" H 1958 5429 50  0000 L CNN
-F 2 "perso:Probing_pad" H 2100 5400 50  0001 C CNN
+F 2 "telec:Probing_pad" H 2100 5400 50  0001 C CNN
 F 3 "~" H 2100 5400 50  0001 C CNN
 	1    1900 5400
@@
 F 0 "TP14" H 1958 6120 50  0000 L CNN
 F 1 "R" H 1958 6029 50  0000 L CNN
-F 2 "perso:Probing_pad" H 2100 6000 50  0001 C CNN
+F 2 "telec:Probing_pad" H 2100 6000 50  0001 C CNN
 F 3 "~" H 2100 6000 50  0001 C CNN
 	1    1900 6000
@@
 $EndComp
 $Comp
-L perso:ADR291GT9Z U02
+L telec:ADR291GT9Z U02
 U 1 1 5C39FFFF
 P 6500 950
@@
 	6900 1400 6900 1350
 $Comp
-L perso:LT1178 U10
+L telec:LT1178 U10
 U 2 1 5C24D302
 P 1550 3600
@@
 F 0 "TP10" H 3308 2670 50  0000 L CNN
 F 1 "Ref" H 3308 2579 50  0000 L CNN
-F 2 "perso:Probing_pad" H 3450 2550 50  0001 C CNN
+F 2 "telec:Probing_pad" H 3450 2550 50  0001 C CNN
 F 3 "~" H 3450 2550 50  0001 C CNN
 	1    3250 2550
@@
 F 0 "TP28" H 10308 1220 50  0000 L CNN
 F 1 "~RDY" H 10308 1129 50  0000 L CNN
-F 2 "perso:Probing_pad" H 10450 1100 50  0001 C CNN
+F 2 "telec:Probing_pad" H 10450 1100 50  0001 C CNN
 F 3 "~" H 10450 1100 50  0001 C CNN
 	1    10250 1100
@@
 F 0 "TP25" H 9208 970 50  0000 L CNN
 F 1 "~ADC_RST" H 9208 879 50  0000 L CNN
-F 2 "perso:Probing_pad" H 9350 850 50  0001 C CNN
+F 2 "telec:Probing_pad" H 9350 850 50  0001 C CNN
 F 3 "~" H 9350 850 50  0001 C CNN
 	1    9150 850
@@
 F 0 "TP21" H 8508 1370 50  0000 L CNN
 F 1 "MISO" H 8508 1279 50  0000 L CNN
-F 2 "perso:Probing_pad" H 8650 1250 50  0001 C CNN
+F 2 "telec:Probing_pad" H 8650 1250 50  0001 C CNN
 F 3 "~" H 8650 1250 50  0001 C CNN
 	1    8450 1250
@@
 F 0 "TP22" H 8758 1570 50  0000 L CNN
 F 1 "MOSI" H 8758 1479 50  0000 L CNN
-F 2 "perso:Probing_pad" H 8900 1450 50  0001 C CNN
+F 2 "telec:Probing_pad" H 8900 1450 50  0001 C CNN
 F 3 "~" H 8900 1450 50  0001 C CNN
 	1    8700 1450
@@
 F 0 "TP23" H 9208 1820 50  0000 L CNN
 F 1 "~ADC_CS" H 9208 1729 50  0000 L CNN
-F 2 "perso:Probing_pad" H 9350 1700 50  0001 C CNN
+F 2 "telec:Probing_pad" H 9350 1700 50  0001 C CNN
 F 3 "~" H 9350 1700 50  0001 C CNN
 	1    9150 1700
@@
 F 0 "TP20" H 8258 1570 50  0000 L CNN
 F 1 "CLK" H 8258 1479 50  0000 L CNN
-F 2 "perso:Probing_pad" H 8400 1450 50  0001 C CNN
+F 2 "telec:Probing_pad" H 8400 1450 50  0001 C CNN
 F 3 "~" H 8400 1450 50  0001 C CNN
 	1    8200 1450
@@
 F 0 "TP29" H 10558 1020 50  0000 L CNN
 F 1 "~SYNC" H 10558 929 50  0000 L CNN
-F 2 "perso:Probing_pad" H 10700 900 50  0001 C CNN
+F 2 "telec:Probing_pad" H 10700 900 50  0001 C CNN
 F 3 "~" H 10700 900 50  0001 C CNN
 	1    10500 900
@@
 F 0 "TP27" H 10058 1020 50  0000 L CNN
 F 1 "~STANDBY" H 10058 929 50  0000 L CNN
-F 2 "perso:Probing_pad" H 10200 900 50  0001 C CNN
+F 2 "telec:Probing_pad" H 10200 900 50  0001 C CNN
 F 3 "~" H 10200 900 50  0001 C CNN
 	1    10000 900
@@
 F 0 "TP24" H 9458 2020 50  0000 L CNN
 F 1 "~SCR_CS" H 9458 1929 50  0000 L CNN
-F 2 "perso:Probing_pad" H 9600 1900 50  0001 C CNN
+F 2 "telec:Probing_pad" H 9600 1900 50  0001 C CNN
 F 3 "~" H 9600 1900 50  0001 C CNN
 	1    9400 1900
@@
 F 0 "TP26" H 9458 1170 50  0000 L CNN
 F 1 "~SCR_RST" H 9458 1079 50  0000 L CNN
-F 2 "perso:Probing_pad" H 9600 1050 50  0001 C CNN
+F 2 "telec:Probing_pad" H 9600 1050 50  0001 C CNN
 F 3 "~" H 9600 1050 50  0001 C CNN
 	1    9400 1050
@@
 F 0 "TP210" H 10058 2020 50  0000 L CNN
 F 1 "D~C" H 10058 1929 50  0000 L CNN
-F 2 "perso:Probing_pad" H 10200 1900 50  0001 C CNN
+F 2 "telec:Probing_pad" H 10200 1900 50  0001 C CNN
 F 3 "~" H 10200 1900 50  0001 C CNN
 	1    10000 1900
